Commit message: Fix joint for fridge door

File: resources/objects/apartment.urdf (robot description, URDF)
Before this commit: robot apartment, 113 links, 112 joints
Joints:
- joint cabinet3_door_top_out_joint: limit lower=0.0 upper=0.02 effort=1.0 velocity=1.5708 -> lower=0.0 upper=1.5708 effort=1.0 velocity=1.5708; type prismatic -> revolute

File: resources/objects/apartment_without_walls.urdf (robot description, URDF)
Before this commit: robot apartment, 106 links, 105 joints
Joints:
- joint cabinet3_door_top_out_joint: limit lower=0.0 upper=0.02 effort=1.0 velocity=1.5708 -> lower=0.0 upper=1.5708 effort=1.0 velocity=1.5708; type prismatic -> revolute
